File: hardware/webasto-mainboard/analog_io.kicad_sch (KiCad schematic)
At the start: 18 parts

Commit message: Update schematics.  Had a better idea.
Other:
- note added: "Need OutdoorTempSensor. Need to change GlowPlug to using a Kelvin 4-wire setup"
Changed lines of the file:
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@@
     (effects (font (size 1.27 1.27)) (justify left bottom))
+  )
+  (text "Need OutdoorTempSensor.\nNeed to change GlowPlug to using a Kelvin 4-wire setup"
+    (at 271.018 75.819 180)
+    (effects (font (size 1.27 1.27)) (justify right bottom))
   )
   (text "/ 4 for max temp of 350C (at 12V)" (at 92.202 66.548 0)

Commit message: More moving of stuff to sensor boards
- not sure I have the glow plug part right quite yet.
Parts:
- removed C?: 1uF, symbol Device:C
- removed C?: 100nF, symbol Device:C
- removed R? (x2): 30k1 1%, symbol Device:R
- removed R? (x2): 49k9 1%, symbol Device:R
- removed R? (x4): 10k0 1%, symbol Device:R
- removed R? (x2): 10k, symbol Device:R
- removed U?: AD7994BRUZ-0REEL, UltraLibrarian:AD7994BRUZ-0REEL, symbol UltraLibrarian:AD7994BRUZ-0REEL
- removed U? (x5): Opamp_Quad, symbol Device:Opamp_Quad
Connections:
- no-connect marks 1 -> 0
Other:
- note removed: "/ 4 for max temp of 125C (at 12V)"
- note removed: "/ 4 for max temp of 350C (at 12V)"
- note removed: "/ 6"
- note removed: "/ 6 to allow for max around 20V"
- note removed: "I2C Address 0x40"
- note removed: "Need OutdoorTempSensor. Need to change GlowPlug to using a Kelvin 4-wire setup"
- note removed: "V = Vin * R2/(R1 + R2) V / Vin = R2/(R1 + R2) 1/4 = R2/(R1 + R2) (R1 + R2)/R2 = 4 R1 = 30k1 1% R2 = 10k0 1%"
- note removed: "V = Vin * R2/(R1 + R2) V / Vin = R2/(R1 + R2) 1/6 = R2/(R1 + R2) (R1 + R2)/R2 = 6 R1 = 49k9 1% R2 = 10k0 1%"
