File: hardware/webasto-mainboard/connectors.kicad_sch (KiCad schematic)
At the start: 7 parts, among them J2 I2C

Commit message: Move start/run to sensor board, add CANBUS
- WiFi is not being very helpful, and I'm concerned it won't work well once
  installed in the bus...  CANBus wiring is easy.
- Removed both Start/Run and the Vehicle Fan Relay from X1 to make space for
  canbus
- moved LEDs onto an I2C gpio extender.
- will need to still plumb in CAN_EN support
- will also need to yank out the WiFi stuff that won't stay stable anyways
  and reroute the CBOR out the CANBus instead of WiFi
- Vehicle Fan control will need to move to a LINBus fan controller board
Connections:
- net StartRun renamed CAN_HI
- net VehicleFanRelay renamed CAN_LO
Changed lines of the file:
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@@
   (title_block
     (title "Webasto Replacement Mainboard (Thermo Top C)")
-    (date "2023-02-22")
+    (date "2023-02-23")
     (rev "2.0")
     (company "Gavin Hurlbut")
@@
     )
   )
+  (global_label "CAN_LO" (shape bidirectional) (at 159.512 58.166 0) (fields_autoplaced)
+    (effects (font (size 1.0922 1.0922)) (justify left))
+    (property "Intersheet References" "${INTERSHEET_REFS}" (id 0) (at 167.6202 58.0978 0)
+      (effects (font (size 1.0922 1.0922)) (justify left) hide)
+    )
+  )
   (global_label "SCL" (shape bidirectional) (at 159.512 60.706 0) (fields_autoplaced)
     (effects (font (size 1.27 1.27)) (justify left))
     (property "Intersheet References" "${INTERSHEET_REFS}" (id 0) (at 165.4327 60.6266 0)
-      (effects (font (size 1.27 1.27)) (justify left) hide)
-    )
-  )
-  (global_label "VehicleFanRelay" (shape input) (at 159.512 58.166 0) (fields_autoplaced)
-    (effects (font (size 1.27 1.27)) (justify left))
-    (property "Intersheet References" "${INTERSHEET_REFS}" (id 0) (at 177.2256 58.0866 0)
       (effects (font (size 1.27 1.27)) (justify left) hide)
     )
@@
     )
   )
-  (global_label "StartRun" (shape input) (at 127.254 58.166 180) (fields_autoplaced)
-    (effects (font (size 1.27 1.27)) (justify right))
-    (property "Intersheet References" "${INTERSHEET_REFS}" (id 0) (at 116.6766 58.0866 0)
-      (effects (font (size 1.27 1.27)) (justify right) hide)
+  (global_label "CAN_HI" (shape bidirectional) (at 127.254 58.166 180) (fields_autoplaced)
+    (effects (font (size 1.0922 1.0922)) (justify right))
+    (property "Intersheet References" "${INTERSHEET_REFS}" (id 0) (at 119.5099 58.0978 0)
+      (effects (font (size 1.0922 1.0922)) (justify right) hide)
     )
   )

Commit message: Rejigger the mainboard to use voltage regulator
Parts:
- F1: footprint Resistor_SMD:R_0603_1608Metric_Pad0.98x0.95mm_HandSolder -> Resistor_SMD:R_1812_4532Metric_Pad1.30x3.40mm_HandSolder; Digikey 18-0603L175SLYRTCT-ND -> F2772CT-ND
Connections:
- net +BATT: now reaches F1.2, JX2.1 (Pin_1)
Other:
- moved on the sheet: JX1

Commit message: Removing KLine and I2C from X1, reattaching the external IOs.
Connections:
- net CAN_HI: now also JX1.4 (Pin_4); no longer JX1.1 (Pin_1)
- net CAN_LO: now also JX1.5 (Pin_5); no longer JX1.4 (Pin_4)
- net SCL: no longer JX1.5 (Pin_5)
- net SDA: no longer JX1.3 (Pin_3)
- net KLine renamed IGNITION_SENSE
- new net START_RUN: JX1.1 (Pin_1)
- new net ~{EMERGENCY_STOP}: JX1.3 (Pin_3)
Changed lines of the file:
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@@
   (title_block
     (title "Webasto Replacement Mainboard (Thermo Top C)")
-    (date "2023-03-04")
+    (date "2023-03-08")
     (rev "2.0")
     (company "Gavin Hurlbut")
@@
     (stroke (width 0) (type default) (color 0 0 0 0))
   )
-  (wire (pts (xy 127.762 55.626) (xy 140.843 55.626))
-    (stroke (width 0) (type default) (color 0 0 0 0))
-  )
   (wire (pts (xy 127.762 50.546) (xy 140.843 50.546))
     (stroke (width 0) (type default) (color 0 0 0 0))
   )
   (wire (pts (xy 141.732 120.015) (xy 141.732 122.682))
+    (stroke (width 0) (type default) (color 0 0 0 0))
+  )
+  (wire (pts (xy 127.762 55.626) (xy 140.843 55.626))
     (stroke (width 0) (type default) (color 0 0 0 0))
   )
@@
     )
   )
+  (global_label "IGNITION_SENSE" (shape output) (at 127.762 53.086 180) (fields_autoplaced)
+    (effects (font (size 1.27 1.27)) (justify right))
+    (property "Intersheet References" "${INTERSHEET_REFS}" (id 0) (at 110.2903 53.0066 0)
+      (effects (font (size 1.27 1.27)) (justify right) hide)
+    )
+  )
   (global_label "CirculationPump" (shape input) (at 133.477 117.475 180) (fields_autoplaced)
     (effects (font (size 1.27 1.27)) (justify right))
     (property "Intersheet References" "${INTERSHEET_REFS}" (id 0) (at 115.461 117.3956 0)
-      (effects (font (size 1.27 1.27)) (justify right) hide)
-    )
-  )
-  (global_label "KLine" (shape bidirectional) (at 127.762 53.086 180) (fields_autoplaced)
-    (effects (font (size 1.27 1.27)) (justify right))
-    (property "Intersheet References" "${INTERSHEET_REFS}" (id 0) (at 120.2084 53.0066 0)
       (effects (font (size 1.27 1.27)) (justify right) hide)
     )
@@
     )
   )
-  (global_label "SDA" (shape bidirectional) (at 127.762 55.626 180) (fields_autoplaced)
-    (effects (font (size 1.27 1.27)) (justify right))
-    (property "Intersheet References" "${INTERSHEET_REFS}" (id 0) (at 121.7808 55.5466 0)
-      (effects (font (size 1.27 1.27)) (justify right) hide)
-    )
-  )
   (global_label "FuelPump" (shape input) (at 160.02 55.626 0) (fields_autoplaced)
     (effects (font (size 1.27 1.27)) (justify left))
@@
     )
   )
-  (global_label "CAN_LO" (shape bidirectional) (at 160.02 50.546 0) (fields_autoplaced)
+  (global_label "CAN_LO" (shape bidirectional) (at 160.02 53.086 0) (fields_autoplaced)
     (effects (font (size 1.0922 1.0922)) (justify left))
-    (property "Intersheet References" "${INTERSHEET_REFS}" (id 0) (at 168.1282 50.4778 0)
+    (property "Intersheet References" "${INTERSHEET_REFS}" (id 0) (at 168.1282 53.0178 0)
       (effects (font (size 1.0922 1.0922)) (justify left) hide)
     )
   )
-  (global_label "SCL" (shape bidirectional) (at 160.02 53.086 0) (fields_autoplaced)
-    (effects (font (size 1.27 1.27)) (justify left))
-    (property "Intersheet References" "${INTERSHEET_REFS}" (id 0) (at 165.9407 53.0066 0)
-      (effects (font (size 1.27 1.27)) (justify left) hide)
+  (global_label "~{EMERGENCY_STOP}" (shape output) (at 127.762 55.626 180) (fields_autoplaced)
+    (effects (font (size 1.27 1.27)) (justify right))
+    (property "Intersheet References" "${INTERSHEET_REFS}" (id 0) (at 108.476 55.5466 0)
+      (effects (font (size 1.27 1.27)) (justify right) hide)
     )
   )
@@
     )
   )
-  (global_label "CAN_HI" (shape bidirectional) (at 127.762 50.546 180) (fields_autoplaced)
-    (effects (font (size 1.0922 1.0922)) (justify right))
-    (property "Intersheet References" "${INTERSHEET_REFS}" (id 0) (at 120.0179 50.4778 0)
-      (effects (font (size 1.0922 1.0922)) (justify right) hide)
+  (global_label "CAN_HI" (shape bidirectional) (at 160.02 50.546 0) (fields_autoplaced)
+    (effects (font (size 1.0922 1.0922)) (justify left))
+    (property "Intersheet References" "${INTERSHEET_REFS}" (id 0) (at 167.7641 50.4778 0)
+      (effects (font (size 1.0922 1.0922)) (justify left) hide)
     )
   )
+  (global_label "START_RUN" (shape output) (at 127.762 50.546 180) (fields_autoplaced)
+    (effects (font (size 1.27 1.27)) (justify right))
+    (property "Intersheet References" "${INTERSHEET_REFS}" (id 0) (at 114.947 50.4666 0)
+      (effects (font (size 1.27 1.27)) (justify right) hide)
+    )
+  )
