File: hardware/webasto-mainboard/glow_plug.kicad_sch (KiCad schematic)
At the start: 25 parts, among them Q11 SSM3J374R, Q12 2N7002, Q13 SUD50P04-08, Q14 SUD50P04-08, Q15 SUD50P04-08, Q16 SUD50P04-08, Q17 SUD50P04-08, Q18 2N7002, Q19 2N7002, U6 LM7805_TO220, U7 INA219BxDCN

Commit message: Move VSYS to ADC2 to avoid the stupid WiFi setup
Parts:
- renumbered R24 to R26, R25 to R27, R26 to R28, R27 to R29, R28 to R30, R29 to R31, R30 to R32, R31 to R33, R32 to R34, R33 to R35
Changed lines of the file:
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@@
   (title_block
     (title "Webasto Replacement Mainboard (Thermo Top C)")
-    (date "2023-02-14")
+    (date "2023-02-22")
     (rev "2.0")
     (company "Gavin Hurlbut")
@@
   (symbol (lib_id "Device:R") (at 120.904 149.225 0) (unit 1)
     (in_bom yes) (on_board yes) (fields_autoplaced)
-    (property "Reference" "R28" (id 0) (at 123.698 147.9549 0)
+    (property "Reference" "R30" (id 0) (at 123.698 147.9549 0)
       (effects (font (size 1.27 1.27)) (justify left))
     )
@@
   (symbol (lib_id "Device:R") (at 74.803 83.312 0) (unit 1)
     (in_bom yes) (on_board yes) (fields_autoplaced)
-    (property "Reference" "R26" (id 0) (at 76.581 82.0419 0)
+    (property "Reference" "R28" (id 0) (at 76.581 82.0419 0)
       (effects (font (size 1.27 1.27)) (justify left))
     )
@@
   (symbol (lib_id "Device:R") (at 88.519 52.07 180) (unit 1)
     (in_bom yes) (on_board yes)
-    (property "Reference" "R27" (id 0) (at 91.059 50.7999 0)
+    (property "Reference" "R29" (id 0) (at 91.059 50.7999 0)
       (effects (font (size 1.27 1.27)) (justify right))
     )
@@
   (symbol (lib_id "Device:R") (at 63.119 52.07 0) (unit 1)
     (in_bom yes) (on_board yes)
-    (property "Reference" "R25" (id 0) (at 65.151 50.7999 0)
+    (property "Reference" "R27" (id 0) (at 65.151 50.7999 0)
       (effects (font (size 1.27 1.27)) (justify left))
     )
@@
   (symbol (lib_id "Device:R") (at 57.785 96.266 90) (unit 1)
     (in_bom yes) (on_board yes) (fields_autoplaced)
-    (property "Reference" "R24" (id 0) (at 57.785 89.662 90))
+    (property "Reference" "R26" (id 0) (at 57.785 89.662 90))
     (property "Value" "10R" (id 1) (at 57.785 92.202 90))
     (property "Footprint" "Resistor_SMD:R_0805_2012Metric_Pad1.20x1.40mm_HandSolder" (id 2) (at 57.785 98.044 90)
@@
   (symbol (lib_id "Device:R") (at 196.977 125.476 0) (mirror x) (unit 1)
     (in_bom yes) (on_board yes) (fields_autoplaced)
-    (property "Reference" "R31" (id 0) (at 194.691 124.2059 0)
+    (property "Reference" "R33" (id 0) (at 194.691 124.2059 0)
       (effects (font (size 1.27 1.27)) (justify right))
     )
@@
   (symbol (lib_id "Device:R") (at 211.709 92.202 180) (unit 1)
     (in_bom yes) (on_board yes) (fields_autoplaced)
-    (property "Reference" "R32" (id 0) (at 214.503 90.9319 0)
+    (property "Reference" "R34" (id 0) (at 214.503 90.9319 0)
       (effects (font (size 1.27 1.27)) (justify right))
     )
@@
   (symbol (lib_id "Device:R") (at 211.709 125.984 180) (unit 1)
     (in_bom yes) (on_board yes) (fields_autoplaced)
-    (property "Reference" "R33" (id 0) (at 214.503 124.7139 0)
+    (property "Reference" "R35" (id 0) (at 214.503 124.7139 0)
       (effects (font (size 1.27 1.27)) (justify right))
     )
@@
   (symbol (lib_id "Device:R") (at 190.119 54.356 0) (mirror x) (unit 1)
     (in_bom yes) (on_board yes) (fields_autoplaced)
-    (property "Reference" "R29" (id 0) (at 187.833 53.0859 0)
+    (property "Reference" "R31" (id 0) (at 187.833 53.0859 0)
       (effects (font (size 1.27 1.27)) (justify right))
     )
@@
   (symbol (lib_id "Device:R") (at 196.977 91.694 0) (mirror x) (unit 1)
     (in_bom yes) (on_board yes) (fields_autoplaced)
-    (property "Reference" "R30" (id 0) (at 194.691 90.4239 0)
-      (effects (font (size 1.27 1.27)) (justify right))
-    )
+    (property "Reference" "R32" (id 0) (at 194.691 90.4239 0)
+      (effects (font (size 1.27 1.27)) (justify right))
+    )

Commit message: Move the LED to the mainboard
- due to how the driver doesn't share the SPI bus well, you currently can
  either use the TCP stack or the GPIOs.  Mixing will cause weird crashes.
- so I'm adding the LED onto the mainboard directly.
Parts:
- renumbered D11 to D12, D12 to D13, R26 to R27, R27 to R28, R28 to R29, R29 to R30, R30 to R31, R31 to R32, R32 to R33, R33 to R34, R34 to R35, R35 to R36
Changed lines of the file:
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@@
   (symbol (lib_name "+3V3_1") (lib_id "power:+3V3") (at 202.565 29.972 0) (unit 1)
     (in_bom yes) (on_board yes) (fields_autoplaced)
-    (property "Reference" "#PWR074" (id 0) (at 202.565 33.782 0)
+    (property "Reference" "#PWR075" (id 0) (at 202.565 33.782 0)
       (effects (font (size 1.27 1.27)) hide)
     )
@@
   (symbol (lib_name "GND_8") (lib_id "power:GND") (at 202.565 58.166 0) (unit 1)
     (in_bom yes) (on_board yes) (fields_autoplaced)
-    (property "Reference" "#PWR075" (id 0) (at 202.565 64.516 0)
+    (property "Reference" "#PWR076" (id 0) (at 202.565 64.516 0)
       (effects (font (size 1.27 1.27)) hide)
     )
@@
   (symbol (lib_id "Device:R") (at 120.904 149.225 0) (unit 1)
     (in_bom yes) (on_board yes) (fields_autoplaced)
-    (property "Reference" "R30" (id 0) (at 123.698 147.9549 0)
+    (property "Reference" "R31" (id 0) (at 123.698 147.9549 0)
       (effects (font (size 1.27 1.27)) (justify left))
     )
@@
   (symbol (lib_id "power:+12V") (at 155.829 53.594 0) (unit 1)
     (in_bom yes) (on_board yes) (fields_autoplaced)
-    (property "Reference" "#PWR069" (id 0) (at 155.829 57.404 0)
+    (property "Reference" "#PWR070" (id 0) (at 155.829 57.404 0)
       (effects (font (size 1.27 1.27)) hide)
     )
@@
   (symbol (lib_id "Device:R") (at 74.803 83.312 0) (unit 1)
     (in_bom yes) (on_board yes) (fields_autoplaced)
-    (property "Reference" "R28" (id 0) (at 76.581 82.0419 0)
+    (property "Reference" "R29" (id 0) (at 76.581 82.0419 0)
       (effects (font (size 1.27 1.27)) (justify left))
     )
@@
   (symbol (lib_id "Device:R") (at 88.519 52.07 180) (unit 1)
     (in_bom yes) (on_board yes)
-    (property "Reference" "R29" (id 0) (at 91.059 50.7999 0)
+    (property "Reference" "R30" (id 0) (at 91.059 50.7999 0)
       (effects (font (size 1.27 1.27)) (justify right))
     )
@@
   (symbol (lib_name "+3V3_2") (lib_id "power:+3V3") (at 196.977 85.344 0) (unit 1)
     (in_bom yes) (on_board yes) (fields_autoplaced)
-    (property "Reference" "#PWR072" (id 0) (at 196.977 89.154 0)
+    (property "Reference" "#PWR073" (id 0) (at 196.977 89.154 0)
       (effects (font (size 1.27 1.27)) hide)
     )
@@
   (symbol (lib_name "GND_2") (lib_id "power:GND") (at 74.803 103.378 0) (unit 1)
     (in_bom yes) (on_board yes) (fields_autoplaced)
-    (property "Reference" "#PWR063" (id 0) (at 74.803 109.728 0)
+    (property "Reference" "#PWR064" (id 0) (at 74.803 109.728 0)
       (effects (font (size 1.27 1.27)) hide)
     )
@@
   (symbol (lib_id "Device:R") (at 63.119 52.07 0) (unit 1)
     (in_bom yes) (on_board yes)
-    (property "Reference" "R27" (id 0) (at 65.151 50.7999 0)
+    (property "Reference" "R28" (id 0) (at 65.151 50.7999 0)
       (effects (font (size 1.27 1.27)) (justify left))
     )
@@
   (symbol (lib_name "+3V3_2") (lib_id "power:+3V3") (at 196.977 119.126 0) (unit 1)
     (in_bom yes) (on_board yes) (fields_autoplaced)
-    (property "Reference" "#PWR073" (id 0) (at 196.977 122.936 0)
+    (property "Reference" "#PWR074" (id 0) (at 196.977 122.936 0)
       (effects (font (size 1.27 1.27)) hide)
     )
@@
   (symbol (lib_id "Device:R") (at 57.785 96.266 90) (unit 1)
     (in_bom yes) (on_board yes) (fields_autoplaced)
-    (property "Reference" "R26" (id 0) (at 57.785 89.662 90))
+    (property "Reference" "R27" (id 0) (at 57.785 89.662 90))
     (property "Value" "10R" (id 1) (at 57.785 92.202 90))
     (property "Footprint" "Resistor_SMD:R_0805_2012Metric_Pad1.20x1.40mm_HandSolder" (id 2) (at 57.785 98.044 90)
@@
   (symbol (lib_id "Diode:BAT54SW") (at 152.4 132.461 270) (mirror x) (unit 1)
     (in_bom yes) (on_board yes) (fields_autoplaced)
-    (property "Reference" "D11" (id 0) (at 154.7368 131.1909 90)
+    (property "Reference" "D12" (id 0) (at 154.7368 131.1909 90)
       (effects (font (size 1.27 1.27)) (justify left))
     )
@@
   (symbol (lib_id "Device:R") (at 196.977 125.476 0) (mirror x) (unit 1)
     (in_bom yes) (on_board yes) (fields_autoplaced)
-    (property "Reference" "R33" (id 0) (at 194.691 124.2059 0)
+    (property "Reference" "R34" (id 0) (at 194.691 124.2059 0)
       (effects (font (size 1.27 1.27)) (justify right))
     )
@@
   (symbol (lib_name "GND_9") (lib_id "power:GND") (at 120.904 157.607 0) (unit 1)
     (in_bom yes) (on_board yes) (fields_autoplaced)
-    (property "Reference" "#PWR066" (id 0) (at 120.904 163.957 0)
+    (property "Reference" "#PWR067" (id 0) (at 120.904 163.957 0)
       (effects (font (size 1.27 1.27)) hide)
     )
@@
   (symbol (lib_name "+12V_3") (lib_id "power:+12V") (at 211.709 85.852 0) (unit 1)
     (in_bom yes) (on_board yes) (fields_autoplaced)
-    (property "Reference" "#PWR076" (id 0) (at 211.709 89.662 0)
+    (property "Reference" "#PWR077" (id 0) (at 211.709 89.662 0)
       (effects (font (size 1.27 1.27)) hide)
     )
@@
   (symbol (lib_name "GND_5") (lib_id "power:GND") (at 88.773 38.1 0) (unit 1)
     (in_bom yes) (on_board yes)
-    (property "Reference" "#PWR064" (id 0) (at 88.773 44.45 0)
+    (property "Reference" "#PWR065" (id 0) (at 88.773 44.45 0)
       (effects (font (size 1.27 1.27)) hide)
     )
@@
   (symbol (lib_id "Device:R") (at 211.709 92.202 180) (unit 1)
     (in_bom yes) (on_board yes) (fields_autoplaced)
-    (property "Reference" "R34" (id 0) (at 214.503 90.9319 0)
+    (property "Reference" "R35" (id 0) (at 214.503 90.9319 0)
       (effects (font (size 1.27 1.27)) (justify right))
     )
@@
   (symbol (lib_id "power:GND") (at 155.829 78.613 0) (unit 1)
     (in_bom yes) (on_board yes) (fields_autoplaced)
-    (property "Reference" "#PWR070" (id 0) (at 155.829 84.963 0)
+    (property "Reference" "#PWR071" (id 0) (at 155.829 84.963 0)
       (effects (font (size 1.27 1.27)) hide)
     )
@@
   (symbol (lib_name "GND_8") (lib_id "power:GND") (at 190.119 60.198 0) (unit 1)
     (in_bom yes) (on_board yes) (fields_autoplaced)
-    (property "Reference" "#PWR071" (id 0) (at 190.119 66.548 0)
+    (property "Reference" "#PWR072" (id 0) (at 190.119 66.548 0)
       (effects (font (size 1.27 1.27)) hide)
     )
@@
   (symbol (lib_name "+12V_2") (lib_id "power:+12V") (at 63.119 27.686 0) (unit 1)
     (in_bom yes) (on_board yes)
-    (property "Reference" "#PWR061" (id 0) (at 63.119 31.496 0)
+    (property "Reference" "#PWR062" (id 0) (at 63.119 31.496 0)
       (effects (font (size 1.27 1.27)) hide)
     )
@@
   (symbol (lib_name "+12V_3") (lib_id "power:+12V") (at 211.709 119.634 0) (unit 1)
     (in_bom yes) (on_board yes) (fields_autoplaced)
-    (property "Reference" "#PWR077" (id 0) (at 211.709 123.444 0)
+    (property "Reference" "#PWR078" (id 0) (at 211.709 123.444 0)
       (effects (font (size 1.27 1.27)) hide)
     )
@@
   (symbol (lib_id "Diode:BAT54SW") (at 155.829 64.008 270) (mirror x) (unit 1)
     (in_bom yes) (on_board yes) (fields_autoplaced)
-    (property "Reference" "D12" (id 0) (at 158.1658 62.7379 90)
+    (property "Reference" "D13" (id 0) (at 158.1658 62.7379 90)
       (effects (font (size 1.27 1.27)) (justify left))
     )
@@
   (symbol (lib_id "power:GND") (at 152.4 145.669 0) (unit 1)
     (in_bom yes) (on_board yes) (fields_autoplaced)
-    (property "Reference" "#PWR068" (id 0) (at 152.4 152.019 0)
+    (property "Reference" "#PWR069" (id 0) (at 152.4 152.019 0)
       (effects (font (size 1.27 1.27)) hide)
     )
@@
   (symbol (lib_id "power:+12V") (at 152.4 122.301 0) (unit 1)
     (in_bom yes) (on_board yes) (fields_autoplaced)
-    (property "Reference" "#PWR067" (id 0) (at 152.4 126.111 0)
+    (property "Reference" "#PWR068" (id 0) (at 152.4 126.111 0)
       (effects (font (size 1.27 1.27)) hide)
     )
@@
   (symbol (lib_name "GND_3") (lib_id "power:GND") (at 63.119 58.674 0) (unit 1)
     (in_bom yes) (on_board yes) (fields_autoplaced)
-    (property "Reference" "#PWR062" (id 0) (at 63.119 65.024 0)
+    (property "Reference" "#PWR063" (id 0) (at 63.119 65.024 0)
       (effects (font (size 1.27 1.27)) hide)
     )
@@
   (symbol (lib_id "Device:R") (at 211.709 125.984 180) (unit 1)
     (in_bom yes) (on_board yes) (fields_autoplaced)
-    (property "Reference" "R35" (id 0) (at 214.503 124.7139 0)
+    (property "Reference" "R36" (id 0) (at 214.503 124.7139 0)
       (effects (font (size 1.27 1.27)) (justify right))
     )
@@
   (symbol (lib_id "Device:R") (at 190.119 54.356 0) (mirror x) (unit 1)
     (in_bom yes) (on_board yes) (fields_autoplaced)
-    (property "Reference" "R31" (id 0) (at 187.833 53.0859 0)
+    (property "Reference" "R32" (id 0) (at 187.833 53.0859 0)
       (effects (font (size 1.27 1.27)) (justify right))
     )
@@
   (symbol (lib_name "+12V_1") (lib_id "power:+12V") (at 103.759 75.692 0) (unit 1)
     (in_bom yes) (on_board yes) (fields_autoplaced)
-    (property "Reference" "#PWR065" (id 0) (at 103.759 79.502 0)
+    (property "Reference" "#PWR066" (id 0) (at 103.759 79.502 0)
       (effects (font (size 1.27 1.27)) hide)
     )
@@
   (symbol (lib_id "Device:R") (at 196.977 91.694 0) (mirror x) (unit 1)
     (in_bom yes) (on_board yes) (fields_autoplaced)
-    (property "Reference" "R32" (id 0) (at 194.691 90.4239 0)
-      (effects (font (size 1.27 1.27)) (justify right))
-    )
+    (property "Reference" "R33" (id 0) (at 194.691 90.4239 0)
+      (effects (font (size 1.27 1.27)) (justify right))
+    )

Commit message: Move start/run to sensor board, add CANBUS
- WiFi is not being very helpful, and I'm concerned it won't work well once
  installed in the bus...  CANBus wiring is easy.
- Removed both Start/Run and the Vehicle Fan Relay from X1 to make space for
  canbus
- moved LEDs onto an I2C gpio extender.
- will need to still plumb in CAN_EN support
- will also need to yank out the WiFi stuff that won't stay stable anyways
  and reroute the CBOR out the CANBus instead of WiFi
- Vehicle Fan control will need to move to a LINBus fan controller board
Parts:
- renumbered D12 to D11, D13 to D12, Q13 to Q10, Q14 to Q11, Q15 to Q12, Q16 to Q13, Q17 to Q14, Q18 to Q15, Q19 to Q16, Q11 to Q8, Q12 to Q9, R27 to R22, R28 to R23, R29 to R24, R30 to R25, R31 to R26, R32 to R27, R33 to R28, R34 to R29, R35 to R30, R36 to R31

Commit message: Moved the INA219 into my own library
Parts:
- U7: symbol Analog_ADC:INA219BxDCN -> Beirdo:INA219BxDCN
Changed lines of the file:
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@@
     (pin "1")
   )
-  (symbol (lib_id "Analog_ADC:INA219BxDCN") (at 202.565 45.466 0) (unit 1)
+  (symbol (lib_id "Beirdo:INA219BxDCN") (at 202.565 45.466 0) (unit 1)
     (in_bom yes) (on_board yes) (fields_autoplaced)
     (property "Reference" "U7" (id 0) (at 204.5844 32.004 0)
