File: hardware/qwiic5v-shifter/qwiic5v-shifter.kicad_pcb (KiCad board)
At the start: 2 copper layers, 28 x 9.9 mm, 15 parts, among them J1 QWIIC Connector, J2 QWIIC Connector, Q1 2N7002, Q2 2N7002, U1 LTC3203BEDD-PBF

Commit message: Move the gates of the level translators to the lowside signal
Connections:
- Q1 pad 1: +3V3 -> SDA3V
- Q2 pad 1: +3V3 -> SCL3V
Routing:
- net SDA3V: track 13.9 -> 10.5 mm, vias 3 -> 2
- net SCL3V: track 7.10 -> 9.00 mm
Other:
- board text added: "v2.0"
Changed lines of the file:
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@@
   (title_block
     (title "QWIIC 5V Shifter")
-    (date "2023-01-31")
-    (rev "1.0")
+    (date "2023-02-05")
+    (rev "2.0")
     (company "Gavin Hurlbut")
   )
@@
     (fp_line (start -0.65 -1.125) (end -0.325 -1.45) (layer "F.Fab") (width 0.1))
     (pad "1" smd roundrect (at -0.9375 -0.95) (size 1.475 0.6) (layers "F.Cu" "F.Paste" "F.Mask") (roundrect_rratio 0.25)
-      (net 1 "+3V3") (pinfunction "G") (pintype "input"))
+      (net 8 "SDA3V") (pinfunction "G") (pintype "input"))
     (pad "2" smd roundrect (at -0.9375 0.95) (size 1.475 0.6) (layers "F.Cu" "F.Paste" "F.Mask") (roundrect_rratio 0.25)
       (net 8 "SDA3V") (pinfunction "S") (pintype "passive"))
@@
     (fp_line (start 0.65 -1.45) (end 0.65 1.45) (layer "F.Fab") (width 0.1))
     (pad "1" smd roundrect (at -0.9375 -0.95) (size 1.475 0.6) (layers "F.Cu" "F.Paste" "F.Mask") (roundrect_rratio 0.25)
-      (net 1 "+3V3") (pinfunction "G") (pintype "input"))
+      (net 9 "SCL3V") (pinfunction "G") (pintype "input"))
     (pad "2" smd roundrect (at -0.9375 0.95) (size 1.475 0.6) (layers "F.Cu" "F.Paste" "F.Mask") (roundrect_rratio 0.25)
       (net 9 "SCL3V") (pinfunction "S") (pintype "passive"))
@@
     (property "Sheetname" "")
     (attr smd)
-    (fp_text reference "R1" (at -0.5 -1.9) (layer "B.SilkS")
+    (fp_text reference "R1" (at -2.9 -0.1) (layer "B.SilkS")
       (effects (font (size 1 1) (thickness 0.15)) (justify mirror))
     )
@@
   (gr_line (start 148 79) (end 120 79) (layer "Edge.Cuts") (width 0.1))
   (gr_line (start 120 88.9) (end 148 88.9) (layer "Edge.Cuts") (width 0.1))
+  (gr_text "v2.0" (at 123.7 79.8) (layer "F.SilkS")
+    (effects (font (size 1 1) (thickness 0.15)))
+  )
   (gr_text "3.3V Side" (at 123.9 88.1) (layer "F.SilkS")
     (effects (font (size 1 1) (thickness 0.15)))
@@
   (segment locked (start 133.800001 83.200001) (end 133.5 82.9) (width 0.25) (layer "F.Cu") (net 1))
   (via (at 135.655924 81.841043) (size 0.8) (drill 0.4) (layers "F.Cu" "B.Cu") (net 1))
-  (via (at 126.8 85.5) (size 0.8) (drill 0.4) (layers "F.Cu" "B.Cu") (net 1))
+  (via (at 125.5 86.5) (size 0.8) (drill 0.4) (layers "F.Cu" "B.Cu") (net 1))
   (via (at 133.5 82.9) (size 0.8) (drill 0.4) (layers "F.Cu" "B.Cu") (net 1))
   (segment (start 133.3 83.1) (end 133.5 82.9) (width 0.25) (layer "B.Cu") (net 1))
-  (segment (start 126 84.7) (end 126.8 85.5) (width 0.25) (layer "B.Cu") (net 1))
+  (segment (start 125.2 86.2) (end 125.5 86.5) (width 0.25) (layer "B.Cu") (net 1))
+  (segment (start 125.2 84.7) (end 125.2 86.2) (width 0.25) (layer "B.Cu") (net 1))
   (segment (start 132 83.1) (end 133.3 83.1) (width 0.25) (layer "B.Cu") (net 1))
-  (segment (start 125.2 84.7) (end 126 84.7) (width 0.25) (layer "B.Cu") (net 1))
   (segment (start 135.655924 81.841043) (end 135.596967 81.9) (width 0.25) (layer "B.Cu") (net 1))
   (segment (start 134.5 81.9) (end 133.5 82.9) (width 0.25) (layer "B.Cu") (net 1))
@@
   (segment (start 123.724999 83.2) (end 122.996475 83.2) (width 0.25) (layer "F.Cu") (net 8))
   (segment (start 123.724999 83.2) (end 126.8 83.2) (width 0.25) (layer "F.Cu") (net 8))
-  (segment (start 126.35 86.45) (end 127.3 86.45) (width 0.25) (layer "F.Cu") (net 8))
-  (segment (start 126.1 86.7) (end 126.35 86.45) (width 0.25) (layer "F.Cu") (net 8))
   (segment (start 121.9 84.296475) (end 121.9 84.6) (width 0.25) (layer "F.Cu") (net 8))
-  (segment (start 126.1 87.3) (end 126.1 86.7) (width 0.25) (layer "F.Cu") (net 8))
+  (segment (start 127.3 83.7) (end 127 83.4) (width 0.25) (layer "F.Cu") (net 8))
   (segment (start 122.996475 83.2) (end 121.9 84.296475) (width 0.25) (layer "F.Cu") (net 8))
+  (segment (start 127.3 84.55) (end 127.3 86.45) (width 0.25) (layer "F.Cu") (net 8))
   (segment (start 126.8 83.2) (end 127 83.4) (width 0.25) (layer "F.Cu") (net 8))
+  (segment (start 127.3 84.55) (end 127.3 83.7) (width 0.25) (layer "F.Cu") (net 8))
   (via (at 127 83.4) (size 0.8) (drill 0.4) (layers "F.Cu" "B.Cu") (net 8))
   (via (at 121.9 84.6) (size 0.8) (drill 0.4) (layers "F.Cu" "B.Cu") (net 8))
-  (via (at 126.1 87.3) (size 0.8) (drill 0.4) (layers "F.Cu" "B.Cu") (net 8))
-  (segment (start 127 83.4) (end 127.524511 83.924511) (width 0.25) (layer "B.Cu") (net 8))
   (segment (start 121.9 84.6) (end 123.1 84.6) (width 0.25) (layer "B.Cu") (net 8))
   (segment (start 123.1 84.6) (end 123.2 84.7) (width 0.25) (layer "B.Cu") (net 8))
-  (segment (start 127.524511 85.875489) (end 126.1 87.3) (width 0.25) (layer "B.Cu") (net 8))
-  (segment (start 127.524511 83.924511) (end 127.524511 85.875489) (width 0.25) (layer "B.Cu") (net 8))
   (segment (start 123.724999 82.199999) (end 127.349999 82.199999) (width 0.25) (layer "F.Cu") (net 9))
   (segment (start 123.724999 82.199999) (end 122.500001 82.199999) (width 0.25) (layer "F.Cu") (net 9))
   (segment (start 127.349999 82.199999) (end 127.4 82.25) (width 0.25) (layer "F.Cu") (net 9))
+  (segment (start 127.4 80.35) (end 127.4 82.25) (width 0.25) (layer "F.Cu") (net 9))
   (segment (start 122.500001 82.199999) (end 121.9 82.8) (width 0.25) (layer "F.Cu") (net 9))
   (via (at 121.9 82.8) (size 0.8) (drill 0.4) (layers "F.Cu" "B.Cu") (net 9))
